Commit message: Update code

File: description/ridgeback_ur5/urdf/ur5_arm_ros2_control.urdf.xacro (robot description, xacro)
@@ -2,4 +2,5 @@
 <robot name="ridgeback_ur5_arm_control" xmlns:xacro="http://www.ros.org/wiki/xacro">
   <xacro:arg name="use_mock_hardware" default="true"/>
+  <xacro:property name="use_mock_hardware" value="$(arg use_mock_hardware)"/>
   <!-- Minimal kinematic chain for ros2_control (joint names match ridgeback_ur5.urdf) -->
   <link name="base_link"/>

Commit message: Update initial_pose

File: description/ridgeback_ur5/urdf/ur5_arm_ros2_control.urdf.xacro (robot description, xacro)
@@ -2,5 +2,9 @@
 <robot name="ridgeback_ur5_arm_control" xmlns:xacro="http://www.ros.org/wiki/xacro">
   <xacro:arg name="use_mock_hardware" default="true"/>
+  <xacro:arg name="initial_pose_file" default=""/>
   <xacro:property name="use_mock_hardware" value="$(arg use_mock_hardware)"/>
+  <xacro:property name="initial_pose_file" value="$(arg initial_pose_file)"/>
+  <xacro:property name="initial_pose" value="${xacro.load_yaml(initial_pose_file)}"/>
+  <xacro:property name="arm_init" value="${initial_pose['arm_joints']}"/>
   <!-- Minimal kinematic chain for ros2_control (joint names match ridgeback_ur5.urdf) -->
   <link name="base_link"/>
@@ -63,25 +67,37 @@
     <joint name="ur_arm_shoulder_pan_joint">
       <command_interface name="position"/>
-      <state_interface name="position"/>
+      <state_interface name="position">
+        <param name="initial_value">${arm_init['ur_arm_shoulder_pan_joint']}</param>
+      </state_interface>
     </joint>
     <joint name="ur_arm_shoulder_lift_joint">
       <command_interface name="position"/>
-      <state_interface name="position"/>
+      <state_interface name="position">
+        <param name="initial_value">${arm_init['ur_arm_shoulder_lift_joint']}</param>
+      </state_interface>
     </joint>
     <joint name="ur_arm_elbow_joint">
       <command_interface name="position"/>
-      <state_interface name="position"/>
+      <state_interface name="position">
+        <param name="initial_value">${arm_init['ur_arm_elbow_joint']}</param>
+      </state_interface>
     </joint>
     <joint name="ur_arm_wrist_1_joint">
       <command_interface name="position"/>
-      <state_interface name="position"/>
+      <state_interface name="position">
+        <param name="initial_value">${arm_init['ur_arm_wrist_1_joint']}</param>
+      </state_interface>
     </joint>
     <joint name="ur_arm_wrist_2_joint">
       <command_interface name="position"/>
-      <state_interface name="position"/>
+      <state_interface name="position">
+        <param name="initial_value">${arm_init['ur_arm_wrist_2_joint']}</param>
+      </state_interface>
     </joint>
     <joint name="ur_arm_wrist_3_joint">
       <command_interface name="position"/>
-      <state_interface name="position"/>
+      <state_interface name="position">
+        <param name="initial_value">${arm_init['ur_arm_wrist_3_joint']}</param>
+      </state_interface>
     </joint>
   </ros2_control>

Commit message: Change use_mock_hardware name to use_fake_hardware

File: description/ridgeback_ur5/urdf/ur5_arm_ros2_control.urdf.xacro (robot description, xacro)
@@ -1,7 +1,7 @@
 <?xml version="1.0"?>
 <robot name="ridgeback_ur5_arm_control" xmlns:xacro="http://www.ros.org/wiki/xacro">
-  <xacro:arg name="use_mock_hardware" default="true"/>
+  <xacro:arg name="use_fake_hardware" default="true"/>
   <xacro:arg name="initial_pose_file" default=""/>
-  <xacro:property name="use_mock_hardware" value="$(arg use_mock_hardware)"/>
+  <xacro:property name="use_fake_hardware" value="$(arg use_fake_hardware)"/>
   <xacro:property name="initial_pose_file" value="$(arg initial_pose_file)"/>
   <xacro:property name="initial_pose" value="${xacro.load_yaml(initial_pose_file)}"/>
@@ -59,5 +59,5 @@
   <ros2_control name="RidgebackUr5ArmSystem" type="system">
     <hardware>
-      <xacro:if value="${use_mock_hardware}">
+      <xacro:if value="${use_fake_hardware}">
         <plugin>mock_components/GenericSystem</plugin>
         <param name="mock_sensor_commands">false</param>
