Commit message: COMMIT TOPIC: Add ZMP stability constraint with runtime wrench/frame support
- Add ZMP kinematics + stability constraint using URDF inertial COM and closed-form ZMP.
- Initialize external wrench to zero in code; update it online from WrenchStamped input.
- Add configurable `zmpWrenchTopic` and `zmpWrenchFrameId` in launch/YAML (ridgeback_ur5 + pr2).
- Transform wrench from arbitrary input frame to EE frame before evaluating ZMP.
- Support `zmpStability.implementation` (`soft` relaxed barrier / `hard` augmented Lagrangian), matching envCollision style.
- Add CoM/ZMP visualization markers (blue COM, purple ZMP).
- Publish `/mobile_manipulator/com` and `/mobile_manipulator/zmp` as PoseStamped in mobile base frame.
- Add RViz displays for `/mobile_manipulator/comZmpMarkers`.
- Add fake wrench publisher tools (`launch/pub_fake_wrench.py`, `launch/fake_wrench.launch.py`).

File: description/ridgeback_ur5/urdf/ridgeback_ur5.urdf (robot description, URDF)
Before this commit: robot ridgeback, 29 links, 28 joints
Links:
- link chassis_link: mass 165.304 -> 10.0
