Commit message: Add TT mode for ur5 launch and modify root link to world link for ur5 urdf

File: description/ur5/urdf/ur5.urdf (robot description, URDF)
Before this commit: robot ur5, 12 links, 11 joints
Links:
- removed link root
- added link world
Joints:
- removed joint root_joint
- added joint world_to_base_joint: type fixed, parent world, child ur_arm_base_link, origin xyz=0 0 0 rpy=0 0 0
